Commit message: fix rotation center

File: src/dashgo/dashgo_description/urdf/dashgobase/base.urdf.xacro (robot description, xacro)
@@ -2,7 +2,7 @@
 <robot name="base" xmlns:xacro="http://ros.org/wiki/xacro">
   <!-- Define a number of dimensions using properties -->
-  <xacro:property name="base_x" value="0.40" />
-  <xacro:property name="base_y" value="0.40" />
-  <xacro:property name="base_length" value="0.20" />
+  <xacro:property name="base_x" value="0.46" />
+  <xacro:property name="base_y" value="0.45" />
+  <xacro:property name="base_length" value="0.13" />
   <xacro:property name="wheel_length" value="0.046" />
   <xacro:property name="wheel_radius" value="0.062" />
@@ -82,10 +82,10 @@
   </link>
   <joint name="base_joint" type="fixed">
-<!--
-    <origin xyz="0 0 0.04" rpy="0 0 0" />
--->
-    <origin xyz="0.0 0 ${base_length/2 - wheel_offset_z}" rpy="0 0 0" />
-    <parent link="base_footprint"/>
-    <child link="base_link" />
+    <!--
+        <origin xyz="0 0 0.04" rpy="0 0 0" />
+    -->
+        <origin xyz="-0.175  0 ${base_length/2 - wheel_offset_z}" rpy="0 0 0" />
+        <parent link="base_footprint"/>
+        <child link="base_link" />
   </joint>
    <!-- Add the drive wheels -->

Commit message: update

File: src/dashgo/dashgo_description/urdf/dashgobase/base.urdf.xacro (robot description, xacro)
@@ -85,5 +85,5 @@
         <origin xyz="0 0 0.04" rpy="0 0 0" />
     -->
-        <origin xyz="-0.175  0 ${base_length/2 - wheel_offset_z}" rpy="0 0 0" />
+        <origin xyz="-0.17  0 ${base_length/2 - wheel_offset_z}" rpy="0 0 0" />
         <parent link="base_footprint"/>
         <child link="base_link" />

Commit message: new stable move

File: src/dashgo/dashgo_description/urdf/dashgobase/base.urdf.xacro (robot description, xacro)
@@ -4,10 +4,15 @@
   <xacro:property name="base_x" value="0.46" />
   <xacro:property name="base_y" value="0.45" />
-  <xacro:property name="base_length" value="0.13" />
-  <xacro:property name="wheel_length" value="0.046" />
-  <xacro:property name="wheel_radius" value="0.062" />
-  <xacro:property name="wheel_offset_x" value="-0.08" />
-  <xacro:property name="wheel_offset_y" value="0.176" />
+  <xacro:property name="base_length" value="0.20" />
+  <!-- <xacro:property name="wheel_length" value="0.046" /> -->
+  <!-- <xacro:property name="wheel_radius" value="0.062" /> -->
+  <xacro:property name="wheel_length" value="0.030" />
+  <xacro:property name="wheel_radius" value="0.050" />
+  <!-- <xacro:property name="wheel_offset_x" value="-0.08" /> -->
+  <!-- <xacro:property name="wheel_offset_y" value="0.176" /> -->
   <xacro:property name="wheel_offset_z" value="-0.038" />
+  <xacro:property name="wheel_offset_x" value="0.160" />
+  <xacro:property name="wheel_offset_y" value="0.150" />
+  <!-- <xacro:property name="wheel_offset_z" value="-0.075" /> -->
   <xacro:property name="PI" value="3.1415926" />
   <!-- define a wheel -->
